File: keyboard.kicad_pcb (KiCad board)
At the start: 2 copper layers, 293.8 x 103.2 mm, 132 parts, among them SW1 SW_Push, U1 ATmega32U4-A, Y1 Crystal_GND24_Small

Commit message: Adding files
Parts:
- added F1: Polyfuse_Small, Fuse:Fuse_1206_3216Metric, B.Cu at (231.0, 153.2)
- added J1: Conn_01x04, Connector_JST:JST_SH_SM04B-SRSS-TB_1x04-1MP_P1.00mm_Horizontal, B.Cu at (232.5, 143.7)
- K_0, K_1, K_10, K_11, K_12, K_15, K_16, K_17, K_18, K_19, K_2, K_20, K_21, K_22, K_23, K_24, K_25, K_26, K_29, K_3, K_30, K_31, K_32, K_33, K_34, K_35, K_36, K_37, K_38, K_39, K_4, K_42, K_43, K_44, K_45, K_46, K_47, K_48, K_49, K_5, K_50, K_51, K_53, K_6, K_7, K_8, K_9: footprint MX_Alps_Hybrid:MX-1U-NoLED -> MX_Only:MXOnly-1U-NoLED
- K_13: footprint MX_Alps_Hybrid:MX-2U-NoLED -> MX_Only:MXOnly-2U-NoLED
- K_14, K_27: footprint MX_Alps_Hybrid:MX-1.5U-NoLED -> MX_Only:MXOnly-1.5U-NoLED
- K_28, K_52: footprint MX_Alps_Hybrid:MX-1.75U-NoLED -> MX_Only:MXOnly-1.75U-NoLED
- K_40, K_41: footprint MX_Alps_Hybrid:MX-2.25U-NoLED -> MX_Only:MXOnly-2.25U-NoLED
- K_54, K_55, K_57, K_58: footprint MX_Alps_Hybrid:MX-1.25U-NoLED -> MX_Only:MXOnly-1.25U-NoLED
- K_56: footprint MX_Alps_Hybrid:MX-7U-NoLED -> MX_Only:MXOnly-7U-ReversedStabilizers-NoLED
- moved R2 53.1 mm to (220.9, 149.0)
- moved R3 51.5 mm to (220.9, 146.4)
- moved SW1 44.0 mm to (246.1, 147.7), turned to 90 degrees
- moved C2 24.6 mm to (169.0, 152.3)
- moved C6 23.4 mm to (165.7, 139.0), turned to 0 degrees
- moved C1 20.0 mm to (182.7, 154.8), turned to 0 degrees
- moved R1 19.3 mm to (188.7, 136.1), turned to 0 degrees
- moved Y1 17.2 mm to (165.5, 143.6), turned to -90 degrees
- moved C4 16.1 mm to (176.6, 135.5)
- moved C7 11.2 mm to (165.5, 148.2), turned to 180 degrees
- moved R4 9.20 mm to (173.5, 153.4), turned to 90 degrees
- moved U1 3.31 mm to (181.1, 144.8), turned to 90 degrees
- moved C5 2.04 mm to (191.1, 149.3), turned to 90 degrees
- moved C3 1.78 mm to (190.6, 140.4), turned to -90 degrees
- moved D_55 1.10 mm to (142.4, 145.2)
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Connections:
- R2 pad 1: D+ -> /D+
- R2 pad 2: Net-(U1-D+) -> /D+
- R3 pad 1: D- -> /D-
- R3 pad 2: Net-(U1-D-) -> /D-
- U1 pad 12: col4 -> row0
- U1 pad 18: col7 -> col0
- U1 pad 19: col8 -> col1
- U1 pad 20: col9 -> col2
- U1 pad 21: col10 -> col3
- U1 pad 22: col12 -> col4
- U1 pad 25: col11 -> col5
- U1 pad 26: col13 -> col6
- U1 pad 27: col14 -> col8
- U1 pad 28: col1 -> col9
- U1 pad 29: col2 -> col10
- U1 pad 3: Net-(U1-D-) -> /D-
- U1 pad 30: col3 -> col11
- U1 pad 31: col5 -> col12
- U1 pad 32: col6 -> col13
- U1 pad 36: unconnected-(U1-PF7-Pad36) -> col14
- U1 pad 37: row4 -> col7
- U1 pad 38: row3 -> row4
- U1 pad 39: row2 -> row3
- U1 pad 4: Net-(U1-D+) -> /D+
- U1 pad 40: row1 -> row2
- U1 pad 41: row0 -> row1
- U1 pad 8: col0 -> unconnected-(U1-PB0-Pad8)
Routing:
- net row0: track 0.00 -> 383.7 mm, vias 0 -> 2
- net row1: track 0.00 -> 339.5 mm, vias 0 -> 2
- net row2: track 0.00 -> 304.8 mm, vias 0 -> 2
- net row4: track 0.00 -> 303.9 mm, vias 0 -> 4
- net row3: track 0.00 -> 269.5 mm, vias 0 -> 2
- net col14: track 0.00 -> 256.4 mm, vias 0 -> 1
- net col13: track 0.00 -> 215.0 mm, vias 0 -> 1
- net col12: track 0.00 -> 213.9 mm, vias 0 -> 1
- net col11: track 0.00 -> 208.5 mm, vias 0 -> 1
- net col0: track 0.00 -> 207.5 mm
- net col1: track 0.00 -> 187.3 mm, vias 0 -> 1
- net col10: track 0.00 -> 175.7 mm, vias 0 -> 1
- net GND: track 0.00 -> 173.4 mm, vias 0 -> 5
- net col2: track 0.00 -> 170.2 mm, vias 0 -> 1
- net col3: track 0.00 -> 166.5 mm, vias 0 -> 1
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- added copper zone on B.Cu, net GND
- added copper zone on F.Cu, net GND
Other:
- board size 293.8 x 103.2 mm -> 293.8 x 103.3 mm
