File: keyboard.kicad_sch (KiCad schematic)
At the start: 132 parts, among them SW1 SW_Push, U1 ATmega32U4-A, Y1 Crystal_GND24_Small

Commit message: Adding files
Parts:
- added F1: Polyfuse_Small, Fuse:Fuse_1206_3216Metric, symbol Device:Polyfuse_Small
- added J1: Conn_01x04, Connector_JST:JST_SH_SM04B-SRSS-TB_1x04-1MP_P1.00mm_Horizontal, symbol Connector_Generic:Conn_01x04
- K_0, K_1, K_10, K_11, K_12, K_15, K_16, K_17, K_18, K_19, K_2, K_20, K_21, K_22, K_23, K_24, K_25, K_26, K_29, K_3, K_30, K_31, K_32, K_33, K_34, K_35, K_36, K_37, K_38, K_39, K_4, K_42, K_43, K_44, K_45, K_46, K_47, K_48, K_49, K_5, K_50, K_51, K_53, K_6, K_7, K_8, K_9: footprint MX_Alps_Hybrid:MX-1U-NoLED -> MX_Only:MXOnly-1U-NoLED
- K_13: footprint MX_Alps_Hybrid:MX-2U-NoLED -> MX_Only:MXOnly-2U-NoLED
- K_14, K_27: footprint MX_Alps_Hybrid:MX-1.5U-NoLED -> MX_Only:MXOnly-1.5U-NoLED
- K_28, K_52: footprint MX_Alps_Hybrid:MX-1.75U-NoLED -> MX_Only:MXOnly-1.75U-NoLED
- K_40, K_41: footprint MX_Alps_Hybrid:MX-2.25U-NoLED -> MX_Only:MXOnly-2.25U-NoLED
- K_54, K_55, K_57, K_58: footprint MX_Alps_Hybrid:MX-1.25U-NoLED -> MX_Only:MXOnly-1.25U-NoLED
- K_56: footprint MX_Alps_Hybrid:MX-7U-NoLED -> MX_Only:MXOnly-7U-ReversedStabilizers-NoLED
Connections:
- net +5V: now also F1.1
- net D+: now also R2.2, U1.4 (D+), J1.2 (Pin_2)
- net D-: now also R3.2, U1.3 (D-), J1.3 (Pin_3)
- net GND: now also J1.4 (Pin_4)
- net col0: now also U1.18 (PD0); no longer U1.8 (PB0)
- net col1: now also U1.19 (PD1); no longer U1.28 (PB4)
- net col10: now also U1.29 (PB5); no longer U1.21 (PD3)
- net col11: now also U1.30 (PB6); no longer U1.25 (PD4)
- net col12: now also U1.31 (PC6); no longer U1.22 (PD5)
- net col13: now also U1.32 (PC7); no longer U1.26 (PD6)
- net col14: now also U1.36 (PF7); no longer U1.27 (PD7)
- net col2: now also U1.20 (PD2); no longer U1.29 (PB5)
- net col3: now also U1.21 (PD3); no longer U1.30 (PB6)
- net col4: now also U1.22 (PD5); no longer U1.12 (PB7)
- net col5: now also U1.25 (PD4); no longer U1.31 (PC6)
- net col6: now also U1.26 (PD6); no longer U1.32 (PC7)
- net col7: now also U1.37 (PF6); no longer U1.18 (PD0)
- net col8: now also U1.27 (PD7); no longer U1.19 (PD1)
- net col9: now also U1.28 (PB4); no longer U1.20 (PD2)
- net row0: now also U1.12 (PB7); no longer U1.41 (PF0)
- net row1: now also U1.41 (PF0); no longer U1.40 (PF1)
- net row2: now also U1.40 (PF1); no longer U1.39 (PF4)
- net row3: now also U1.39 (PF4); no longer U1.38 (PF5)
- net row4: now also U1.38 (PF5); no longer U1.37 (PF6)
- new net VCC: F1.2, J1.1 (Pin_1)
- no-connect marks 3 -> 6
Other:
- moved on the sheet: K_0
